File: PlastiSense_PCB/PlastiSense.kicad_pcb (KiCad board)
At the start: 2 copper layers, 15 parts, among them J1 OLED, SW1 SW_Push, SW2 SW_Push, U1 MOUDLE-SEEEDUINO-XIAO-ESP32C3, U2 HALL SENSOR

Commit message: updated
Parts:
- removed D2: LED_Small, LED_SMD:LED_0201_0603Metric_Pad0.64x0.40mm_HandSolder
- removed J1: OLED, Connector_PinSocket_1.00mm:PinSocket_1x04_P1.00mm_Vertical
- removed R4: 220, Resistor_SMD:R_0201_0603Metric_Pad0.64x0.40mm_HandSolder
- removed SW1: SW_Push, Button_Switch_SMD:SW_DIP_SPSTx01_Slide_6.7x4.1mm_W6.73mm_P2.54mm_LowProfile_JPin
- added D3: CLV1L-FKB, LED_SMD:LED_Cree-PLCC4_3.2x2.8mm_CCW, F.Cu at (146.0, 69.6)
- added J2: Conn_01x04, Connector_PinHeader_1.00mm:PinHeader_1x04_P1.00mm_Vertical, F.Cu at (120.2, 81.2)
- added R5: 220, Resistor_SMD:R_0201_0603Metric_Pad0.64x0.40mm_HandSolder, F.Cu at (149.6, 72.0)
- added R6: 220, Resistor_SMD:R_0201_0603Metric_Pad0.64x0.40mm_HandSolder, F.Cu at (146.8, 74.5)
- added R7: 220, Resistor_SMD:R_0201_0603Metric_Pad0.64x0.40mm_HandSolder, F.Cu at (144.3, 74.5)
- BZ1: footprint Buzzer_Beeper:Buzzer_D14mm_H7mm_P10mm -> Buzzer_Beeper:Buzzer_CUI_CPT-9019S-SMT
- R3: value 220 -> 1k
- SW2: footprint Button_Switch_SMD:SW_Push_1P1T_NO_CK_PTS125Sx85SMTR -> Button_Switch_SMD:SW_SPST_B3U-1000P
- moved H1 100.5 mm to (110.5, 64.7)
- moved C1 100.4 mm to (118.4, 67.0), turned to 180 degrees
- moved R2 95.4 mm to (118.6, 72.0)
- moved R3 95.2 mm to (118.6, 74.5)
- moved U2 90.5 mm to (119.0, 63.4), turned to 180 degrees
- moved BZ1 81.6 mm to (111.8, 74.0)
- moved D1 67.6 mm to (152.2, 67.8), turned to -90 degrees
- moved R1 62.9 mm to (152.2, 71.3), turned to 90 degrees
- moved H2 59.2 mm to (152.5, 78.7)
- moved SW2 52.1 mm to (148.0, 63.8)
- moved U1 33.6 mm to (122.8, 81.9)
Connections:
- R1 pad 1: Net-(R1-Pad1) -> +5V
- U1 pad 1: /H_OUT -> /HALL_OUT
- U1 pad 10: unconnected-(U1-PA5_A9_D9_MISO-Pad10) -> /G_LED
- U1 pad 11: unconnected-(U1-PA6_A10_D10_MOSI-Pad11) -> /B_LED
- U1 pad 2: /B_LED -> unconnected-(U1-PA4_A1_D1-Pad2)
- U1 pad 9: unconnected-(U1-PA7_A8_D8_SCK-Pad9) -> /R_LED
Routing:
- net +5V: track 0.00 -> 53.9 mm, vias 0 -> 3
- net /HALL_OUT: track 0.00 -> 33.5 mm, vias 0 -> 2
- net Net-(BZ1-+): track 0.00 -> 14.9 mm, vias 0 -> 2
- net GND: track 0.00 -> 13.0 mm, vias 0 -> 6
- net +3.3V: track 0.00 -> 11.7 mm, vias 0 -> 2
- net /B_LED: track 0.00 -> 11.0 mm, vias 0 -> 2
- net /SCK: track 0.00 -> 10.2 mm
- net Net-(U2-OUT): track 0.00 -> 9.32 mm
- net /BUZZ: track 0.00 -> 9.05 mm
- net /G_LED: track 0.00 -> 7.93 mm, vias 0 -> 2
- net /SCL: track 0.00 -> 7.09 mm
- net Net-(D3-BK): track 0.00 -> 5.51 mm
- net /R_LED: track 0.00 -> 5.30 mm
- net Net-(D3-RK): track 0.00 -> 4.21 mm
- net Net-(D3-GK): track 0.00 -> 4.21 mm
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- added copper zone on In2.Cu, net +3.3V
- added copper zone on B.Cu, net GND
- added copper zone on F.Cu, net GND
- added copper zone on In1.Cu, net GND
Other:
- board outline added: 50 x 22 mm
- copper layers 2 -> 4
- board text added: "v1.0 PlastiSense"
