File: PlastiSense_PCB/PlastiSense.kicad_sch (KiCad schematic)
At the start: 17 parts, among them J1 OLED, SW1 SW_Push, SW2 SW_Push, U1 MOUDLE-SEEEDUINO-XIAO-ESP32C3, U2 HALL SENSOR

Commit message: updated
Parts:
- removed D2: LED_Small, LED_SMD:LED_0201_0603Metric_Pad0.64x0.40mm_HandSolder, symbol Device:LED_Small
- removed H3, H4: MountingHole, MountingHole:MountingHole_3.2mm_M3, symbol Mechanical:MountingHole
- removed J1: OLED, Connector_PinSocket_1.00mm:PinSocket_1x04_P1.00mm_Vertical, symbol Connector_Generic_MountingPin:Conn_01x04_MountingPin
- removed R4: 220, Resistor_SMD:R_0201_0603Metric_Pad0.64x0.40mm_HandSolder, symbol Device:R_Small
- removed SW1: SW_Push, Button_Switch_SMD:SW_DIP_SPSTx01_Slide_6.7x4.1mm_W6.73mm_P2.54mm_LowProfile_JPin, symbol Switch:SW_Push
- added D3: CLV1L-FKB, LED_SMD:LED_Cree-PLCC4_3.2x2.8mm_CCW, symbol LED:CLV1L-FKB
- added J2: Conn_01x04, Connector_PinHeader_1.00mm:PinHeader_1x04_P1.00mm_Vertical, symbol Connector_Generic:Conn_01x04
- added R5, R6, R7: 220, Resistor_SMD:R_0201_0603Metric_Pad0.64x0.40mm_HandSolder, symbol Device:R_Small
- BZ1: footprint Buzzer_Beeper:Buzzer_D14mm_H7mm_P10mm -> Buzzer_Beeper:Buzzer_CUI_CPT-9019S-SMT
- R3: value 220 -> 1k
- SW2: footprint Button_Switch_SMD:SW_Push_1P1T_NO_CK_PTS125Sx85SMTR -> Button_Switch_SMD:SW_SPST_B3U-1000P
Connections:
- net H_OUT is gone; now on net HALL_OUT: U1.1 (PA02_A0_D0)
- net +3.3V: now also D3.1 (A)
- net +5V: now also R1.1, J2.3 (Pin_3)
- net B_LED: now also U1.11 (PA6_A10_D10_MOSI), R5.2; no longer U1.2 (PA4_A1_D1)
- net GND: now also J2.4 (Pin_4)
- net SCK: now also J2.2 (Pin_2)
- net SCL: now also J2.1 (Pin_1)
- net G_LED: now reaches U1.10 (PA5_A9_D9_MISO)
- net G_LED: now also R6.2
- net R_LED: now reaches U1.9 (PA7_A8_D8_SCK)
- net R_LED: now also R7.2
- new net: D3.4 (BK), R5.1
- new net: D3.2 (RK), R7.1
- new net: D3.3 (GK), R6.1
- no-connect marks 6 -> 4
Other:
- note added: "POWER LED"
- note removed: "POWER CIRCUIT"
- moved on the sheet: H1, H2
